Commit message: clean up

File: manta_description/urdf/manta_actuators.xacro (robot description, xacro)
@@ -1,7 +1,7 @@
 <?xml version="1.0"?>
-<!--
-     Written by Kristoffer Rakstad Solberg, Student
-     Copyright (c) 2019 Manta AUV, Vortex NTNU.
-     All rights reserved. -->
+<!-- Copyright (c) 2016 The UUV Simulator Authors.
+     All rights reserved.
+     Contributed by Kristoffer Rakstad Solberg,
+     Student2019 Manta AUV, Vortex NTNU. -->
 <robot xmlns:xacro="http://www.ros.org/wiki/xacro">
 <!-- Here you can put in whatever kind of model you want and it will
@@ -11,4 +11,6 @@
   <!-- <xacro:property name="prop_mesh_file" value="file://$(find manta_description)/mesh/manipulator_claw.dae"/> -->
   <!-- Thruster joint and link snippet -->
+<!-- Time constant for thruster dynamics: rpm = K / (Ts + 1)
+    <rotorConstant> T200, 12V for a 2nd order curve fit: tau = gain * abs(x)*x -->
   <xacro:macro name="thruster_macro"
     params="namespace thruster_id *origin">
@@ -17,9 +19,11 @@
       thruster_id="${thruster_id}"
       mesh_filename="${prop_mesh_file_cw}"
-      dyn_time_constant="0.05"
-      rotor_constant="1.0">
+      dyn_time_constant="0.2"
+      rotor_constant="0.000004">
       <xacro:insert_block name="origin"/>
     </xacro:thruster_module_first_order_basic_fcn_macro>
   </xacro:macro>
+<!-- Time constant for thruster dynamics: rpm = K / (Ts + 1)
+    <rotorConstant> T200, 12V for a 2nd order curve fit: tau = gain * abs(x)*x -->
   <xacro:macro name="thruster_macro_ccw"
     params="namespace thruster_id *origin">
@@ -28,6 +32,6 @@
       thruster_id="${thruster_id}"
       mesh_filename="${prop_mesh_file_ccw}"
-      dyn_time_constant="0.05"
-      rotor_constant="1.0">
+      dyn_time_constant="0.2"
+      rotor_constant="0.000004">
       <xacro:insert_block name="origin"/>
     </xacro:thruster_module_first_order_basic_fcn_macro>

File: manta_description/urdf/manta_base.xacro (robot description, xacro)
@@ -1,7 +1,7 @@
 <?xml version="1.0"?>
-<!--
-     Written by Kristoffer Rakstad Solberg, Student
-     Copyright (c) 2019 Manta AUV, Vortex NTNU.
-     All rights reserved. -->
+<!-- Copyright (c) 2016 The UUV Simulator Authors.
+     All rights reserved.
+     Contributed by Kristoffer Rakstad Solberg,
+     Student2019 Manta AUV, Vortex NTNU. -->
 <robot xmlns:xacro="http://www.ros.org/wiki/xacro">
   <!--
@@ -22,5 +22,5 @@
   -->
   <!-- Mass -->
-  <xacro:property name="mass" value="19.0"/>
+  <xacro:property name="mass" value="16.6"/>
   <!-- Describing the dimensions of the vehicle's bounding box: width, length, height -->
   <xacro:property name="x_size" value="0.448"/>
@@ -31,5 +31,5 @@
   <xacro:property name="volume" value="0.01854"/>
   <!-- Center of gravity -->
-  <xacro:property name="cog" value="0 0 -0.03"/>
+  <xacro:property name="cog" value="0 0 -0.08"/>
   <!--
   Center of buoyancy according to eq. (3.1) p. 28 in Berg2012.
@@ -59,6 +59,4 @@
           <mass value="${mass}" />
           <origin xyz="${cog}" rpy="0 0 0"/>
-           <!-- ixx="${0.80947}" ixy="-0.00308" ixz="-0.01546"
-            iyy="${0.87794}" iyz="0.06283" izz="${1.57147}" />  -->
           <inertia
             ixx="${0.503217}" ixy="${0.000204}" ixz="${-0.000526}"

File: manta_description/urdf/manta_gazebo.xacro (robot description, xacro)
@@ -1,7 +1,7 @@
 <?xml version="1.0"?>
-<!--
-     Written by Kristoffer Rakstad Solberg, Student
-     Copyright (c) 2019 Manta AUV, Vortex NTNU.
-     All rights reserved. -->
+<!-- Copyright (c) 2016 The UUV Simulator Authors.
+     All rights reserved.
+     Contributed by Kristoffer Rakstad Solberg,
+     Student2019 Manta AUV, Vortex NTNU. -->
 <robot xmlns:xacro="http://www.ros.org/wiki/xacro">
   <xacro:macro name="manta_hydro_model" params="namespace">
@@ -31,10 +31,10 @@
           <!-- Added mass: see p.28 in Berg2012 -->
           <added_mass>
-            1.7182 0 0 0 0 0
-            0 0 0 0 0 0
-            0 0 5.468 0 0 0
-            0 0 0 10 0 0
-            0 0 0 0 10.2481 0
-            0 0 0 0 0 0.4006
+            10.7727 0 0 0 0 0
+            0 10.7727 0 0 0 0
+            0 0 49.7679 0 0 0
+            0 0 0 1.0092 0 0
+            0 0 0 0 1.0092 0
+            0  0  0  0  0  0
           </added_mass>
           <!--
@@ -44,5 +44,5 @@
           -->
           <linear_damping>
-            -11.7391 -20 -31.8678 -25 -44.9085 -5
+            -9.5909 -9.5909 -42.5798 -13.3040 -13.2181 -1.1559
           </linear_damping>
           <!--
@@ -61,5 +61,5 @@
           -->
           <quadratic_damping>
-            0 0 0 0 0 0
+            -5.1386 -5.1386 -26.1105 0 0 0
           </quadratic_damping>
           <!--

File: uuv_gazebo_plugins/uuv_gazebo_ros_plugins/urdf/thruster_snippets.xacro (robot description, xacro)
@@ -83,5 +83,5 @@
     </joint>
     <link name="${namespace}/thruster_${thruster_id}">
-      <xacro:box_inertial x="0" y="0" z="0" mass="0.001">
+      <xacro:box_inertial x="0.1" y="0.1" z="0.1" mass="0.3">
         <origin xyz="0 0 0" rpy="0 0 0"/>
       </xacro:box_inertial>
