Commit message: changed mass

File: manta_description/urdf/manta_base.xacro (robot description, xacro)
@@ -22,12 +22,12 @@
   -->
   <!-- Mass -->
-  <xacro:property name="mass" value="16.6"/>
+  <xacro:property name="mass" value="30.9"/>
   <!-- Describing the dimensions of the vehicle's bounding box: width, length, height -->
-  <xacro:property name="x_size" value="0.448"/>
-  <xacro:property name="y_size" value="0.444"/>
-  <xacro:property name="z_size" value="0.28066"/>
+  <xacro:property name="x_size" value="0.400"/>
+  <xacro:property name="y_size" value="0.400"/>
+  <xacro:property name="z_size" value="0.20066"/>
   <!-- minion_usv_height is not really! It's just for run... We need first calculate the Fossen parameters -->
   <!-- Volume -->
-  <xacro:property name="volume" value="0.01854"/>
+  <xacro:property name="volume" value="0.0325"/>
   <!-- Center of gravity -->
   <xacro:property name="cog" value="0 0 -0.08"/>

File: manta_description/urdf/manta_gazebo.xacro (robot description, xacro)
@@ -9,5 +9,5 @@
     <link name="${namespace}/base_link">
       <!-- This flag will make the link neutrally buoyant -->
-      <neutrally_buoyant>0</neutrally_buoyant>
+      <neutrally_buoyant>0.0</neutrally_buoyant>
       <!-- Link's volume -->
       <volume>${volume}</volume>

Commit message: changed manta dynamics and world

File: manta_description/urdf/manta_base.xacro (robot description, xacro)
@@ -22,5 +22,5 @@
   -->
   <!-- Mass -->
-  <xacro:property name="mass" value="30.9"/>
+  <xacro:property name="mass" value="30.7"/>
   <!-- Describing the dimensions of the vehicle's bounding box: width, length, height -->
   <xacro:property name="x_size" value="0.400"/>

File: manta_description/urdf/manta_sensors.xacro (robot description, xacro)
@@ -19,4 +19,8 @@
     <origin xyz="-1.32 0 0.8" rpy="0 0 0"/>
   </xacro:default_rpt> -->
+  <!-- Forward-looking sonar sensor
+  <xacro:forward_multibeam_p900 namespace="${namespace}" parent_link="${namespace}/base_link">
+    <origin xyz="0.29 0 -0.06" rpy="0 0 0"/>
+  </xacro:forward_multibeam_p900> -->
   <!-- Pressure  -->
   <xacro:default_pressure_macro namespace="${namespace}" parent_link="${namespace}/base_link">

Commit message: changed dynamics

File: manta_description/urdf/manta_base.xacro (robot description, xacro)
@@ -22,5 +22,5 @@
   -->
   <!-- Mass -->
-  <xacro:property name="mass" value="30.7"/>
+  <xacro:property name="mass" value="30.9"/>
   <!-- Describing the dimensions of the vehicle's bounding box: width, length, height -->
   <xacro:property name="x_size" value="0.400"/>
