Commit message: Move DVL down a bit

File: manta_description/urdf/manta_sensors.xacro (robot description, xacro)
@@ -10,5 +10,5 @@
     parent_link="${namespace}/base_link"
     inertial_reference_frame="${inertial_reference_frame}">
-    <origin xyz="0 0 0" rpy="0 ${0.5*pi} 0"/>
+    <origin xyz="0 0 -0.05" rpy="0 ${0.5*pi} 0"/>
   </xacro:default_dvl_macro>
   <!-- Magnetometer  -->
