Commit message: Change gladlaks namespace to beluga, still some random things using a manta namespace, will be fixed in the future. Changed DVL and frontcamera to match Beluga.

File: beluga_description/robots/beluga_default.xacro (robot description, xacro)
@@ -17,8 +17,8 @@
   <xacro:arg name="inertial_reference_frame" default="world"/>
   <!-- Include the ROV macro file -->
-  <xacro:include filename="$(find gladlaks_description)/urdf/gladlaks_base.xacro"/>
+  <xacro:include filename="$(find beluga_description)/urdf/beluga_base.xacro"/>
   <xacro:include filename="$(find manta_description)/urdf/manta_gazebo.xacro"/>
   <!-- Create the rexrov -->
-  <xacro:gladlaks_base
+  <xacro:beluga_base
     namespace="$(arg namespace)"
     inertial_reference_frame="$(arg inertial_reference_frame)">
@@ -34,5 +34,5 @@
       </plugin>
     </gazebo>
-  </xacro:gladlaks_base>
+  </xacro:beluga_base>
   <!-- Joint state publisher plugin -->
   <xacro:default_joint_state_publisher namespace="$(arg namespace)" update_rate="50"/>

File: beluga_description/urdf/beluga_actuators.xacro (robot description, xacro)
@@ -7,7 +7,7 @@
 <!-- Here you can put in whatever kind of model you want and it will
   still function as a propeller                                      -->
-  <xacro:property name="prop_mesh_file_cw" value="file://$(find gladlaks_description)/mesh/t200_propccw.dae"/>
-  <xacro:property name="prop_mesh_file_ccw" value="file://$(find gladlaks_description)/mesh/t200_propcw.dae"/>
-  <!-- <xacro:property name="prop_mesh_file" value="file://$(find gladlaks_description)/mesh/manipulator_claw.dae"/> -->
+  <xacro:property name="prop_mesh_file_cw" value="file://$(find beluga_description)/mesh/t200_propccw.dae"/>
+  <xacro:property name="prop_mesh_file_ccw" value="file://$(find beluga_description)/mesh/t200_propcw.dae"/>
+  <!-- <xacro:property name="prop_mesh_file" value="file://$(find beluga_description)/mesh/manipulator_claw.dae"/> -->
   <!-- Thruster joint and link snippet -->
 <!-- Time constant for thruster dynamics: rpm = K / (Ts + 1)

File: beluga_description/urdf/beluga_base.xacro (robot description, xacro)
@@ -47,7 +47,7 @@
   -->
   <!-- Parameters -->
-  <xacro:property name="namespace" value="gladlaks"/>
-  <xacro:property name="visual_mesh_file" value="file://$(find gladlaks_description)/mesh/Gladlaks_centered_body.dae"/>
-  <xacro:macro name="gladlaks_base" params="namespace *gazebo inertial_reference_frame">
+  <xacro:property name="namespace" value="beluga"/>
+  <xacro:property name="visual_mesh_file" value="file://$(find beluga_description)/mesh/beluga_centered_body.dae"/>
+  <xacro:macro name="beluga_base" params="namespace *gazebo inertial_reference_frame">
    <!-- Rigid body description of the base link -->
     <link name="${namespace}/base_link">
@@ -93,10 +93,10 @@
     receive topics on all its thrusters. The robot will not move just by launching
     this file alone -->
-  <xacro:include filename="$(find gladlaks_description)/urdf/gladlaks_actuators.xacro"/>
+  <xacro:include filename="$(find beluga_description)/urdf/beluga_actuators.xacro"/>
    <!-- Publishes -->
    <!-- ONLY NEED FOR SIMULATIONS (GAZEBO SPECIFIC)
      This .xacro file has to run to be able to move the robot when controller
      commands have been sent to the thrusters-->
-  <xacro:include filename="$(find gladlaks_description)/urdf/manta_sensors.xacro"/>
+  <xacro:include filename="$(find beluga_description)/urdf/manta_sensors.xacro"/>
   </xacro:macro>
   <gazebo reference="${namespace}/base_link">

File: beluga_description/urdf/manta_gazebo.xacro (robot description, xacro)
@@ -5,5 +5,5 @@
      Student2019 Manta AUV, Vortex NTNU. -->
 <robot xmlns:xacro="http://www.ros.org/wiki/xacro">
-  <xacro:macro name="gladlaks_hydro_model" params="namespace">
+  <xacro:macro name="beluga_hydro_model" params="namespace">
     <!-- List of hydrodynamic models this robot's links -->
     <link name="${namespace}/base_link">

File: beluga_description/urdf/manta_sensors.xacro (robot description, xacro)
@@ -10,5 +10,5 @@
     parent_link="${namespace}/base_link"
     inertial_reference_frame="${inertial_reference_frame}">
-    <origin xyz="0 0 0" rpy="0 ${0.5*pi} 0"/>
+    <origin xyz="0.074 -0.015 -0.115" rpy="-3.14 1.57 -3.14"/>
   </xacro:default_dvl_macro>
   <!-- Magnetometer  -->
@@ -36,5 +36,5 @@
   <!-- Mount a camera -->
   <xacro:default_camera namespace="${namespace}" parent_link="${namespace}/base_link" suffix="front">
-    <origin xyz="0.29 0.0 0." rpy="0 0 0"/>
+    <origin xyz="0.349 0.0 0.058" rpy="0.01 0.18 -0.005"/>
   </xacro:default_camera>
   <xacro:default_camera namespace="${namespace}" parent_link="${namespace}/base_link" suffix="under">
