Commit message: Update sensor plugins
Signed-off-by: Christopher Strøm <detoxte@gmail.com>

File: uuv_gazebo_plugins/uuv_gazebo_ros_plugins/urdf/thruster_snippets.xacro (robot description, xacro)
@@ -83,5 +83,5 @@
     </joint>
     <link name="${namespace}/thruster_${thruster_id}">
-      <xacro:box_inertial x="0.1" y="0.1" z="0.1" mass="0.3">
+      <xacro:box_inertial x="0" y="0" z="0" mass="0.001">
         <origin xyz="0 0 0" rpy="0 0 0"/>
       </xacro:box_inertial>
@@ -102,5 +102,5 @@
     </link>
     <gazebo>
-      <plugin name="${namespace}_${thruster_id}_thruster_model" filename="libthruster_ros_plugin.so">
+      <plugin name="${namespace}_${thruster_id}_thruster_model" filename="libuuv_thruster_ros_plugin.so">
         <linkName>${namespace}/thruster_${thruster_id}</linkName>
         <jointName>${namespace}/thruster_${thruster_id}_joint</jointName>
@@ -110,8 +110,6 @@
       </plugin>
     </gazebo>
-   <!-- Choose thruster color -->
     <gazebo reference="${namespace}/thruster_${thruster_id}">
       <selfCollide>false</selfCollide>
-    <material>Gazebo/Red</material>
     </gazebo>
   </xacro:macro>

File: uuv_sensor_plugins/uuv_sensor_ros_plugins/urdf/dvl_snippets.xacro (robot description, xacro)
@@ -29,7 +29,7 @@
       update_rate="7"
       topic="dvl"
-      noise_sigma="0.0"
-      noise_amplitude="0.0"
-      scale="0.5">
+      noise_sigma="0"
+      noise_amplitude="0"
+      scale="1">
       <xacro:insert_block name="origin" />
     </xacro:dvl_plugin_macro>
@@ -52,6 +52,4 @@
   </xacro:macro>
   <!-- DEPRECATED MACRO: See default_dvl_sensor_enu -->
-<!--  noise_sigma="1.0"
-      noise_amplitude="1.0" -->
   <xacro:macro name="default_dvl" params="namespace parent_link *origin">
     <xacro:dvl_plugin_macro
@@ -62,11 +60,11 @@
       update_rate="7"
       topic="dvl"
-      noise_sigma="0.0"
-      noise_amplitude="0.0"
-      scale="0.5">
+      noise_sigma="0"
+      noise_amplitude="0"
+      scale="1">
       <xacro:insert_block name="origin" />
     </xacro:dvl_plugin_macro>
   </xacro:macro>
-  <xacro:macro name="dvl_single_sonar" params="namespace suffix index pitch yaw">
+  <xacro:macro name="dvl_single_sonar" params="namespace suffix index pitch yaw update_rate">
     <link name="${namespace}/dvl${suffix}_sonar${index}_link">
       <inertial>
@@ -87,5 +85,5 @@
       <sensor type="ray" name="dvl${suffix}_sonar${index}">
         <pose>0 0 0 0 0 0</pose>
-        <update_rate>1</update_rate>
+        <update_rate>${update_rate}</update_rate>
         <visualize>false</visualize>
         <ray>
@@ -113,5 +111,5 @@
           <gaussianNoise>0.005</gaussianNoise>
           <alwaysOn>true</alwaysOn>
-          <updateRate>1</updateRate>
+          <updateRate>${update_rate}</updateRate>
           <topicName>${topic}_sonar${index}</topicName>
           <frameName>${namespace}/dvl${suffix}_sonar${index}_link</frameName>
@@ -147,23 +145,22 @@
     <xacro:dvl_single_sonar
       namespace="${namespace}" suffix=""
-      index="0" pitch="-0.52" yaw="0.0">
+      index="0" pitch="-0.52" yaw="0.0" update_rate="${update_rate}">
     </xacro:dvl_single_sonar>
     <xacro:dvl_single_sonar
       namespace="${namespace}" suffix=""
-      index="1" pitch="0" yaw="0.52">
+      index="1" pitch="0" yaw="0.52" update_rate="${update_rate}">
     </xacro:dvl_single_sonar>
     <xacro:dvl_single_sonar
       namespace="${namespace}" suffix=""
-      index="2" pitch="0.52" yaw="0.0">
+      index="2" pitch="0.52" yaw="0.0" update_rate="${update_rate}">
     </xacro:dvl_single_sonar>
     <xacro:dvl_single_sonar
       namespace="${namespace}" suffix=""
-      index="3" pitch="0.0" yaw="-0.52">
+      index="3" pitch="0.0" yaw="-0.52" update_rate="${update_rate}">
     </xacro:dvl_single_sonar>
     <gazebo>
       <plugin filename="libuuv_gazebo_ros_dvl_plugin.so" name="libuuv_gazebo_dvl${suffix}_plugin">
         <robot_namespace>${namespace}</robot_namespace> <!-- (string, required): ros namespace in which the messages are published -->
-	<!-- Changed from dvl_link to base_link to get ENU coordinate frame -->
-        <link_name>${namespace}/base_link</link_name> <!-- (string, required): name of the body which holds the IMU sensor -->
+        <link_name>${namespace}/dvl${suffix}_link</link_name> <!-- (string, required): name of the body which holds the IMU sensor -->
         <sensor_topic>${topic}</sensor_topic> <!-- (string): name of the sensor output topic and prefix of service names -->
         <update_rate>${update_rate}</update_rate> <!-- Update period [s] -->

File: uuv_sensor_plugins/uuv_sensor_ros_plugins/urdf/pressure_snippets.xacro (robot description, xacro)
@@ -69,5 +69,5 @@
       <visual>
         <geometry>
-          <mesh filename="file://$(find uuv_sensor_ros_plugins)/meshes/pressure.dae" scale="0.1 0.1 0.1"/>
+          <mesh filename="file://$(find uuv_sensor_ros_plugins)/meshes/pressure.dae" scale="1 1 1"/>
         </geometry>
       </visual>
