Commit message: Fix beluga physics
Signed-off-by: Christopher Strøm <detoxte@gmail.com>

File: beluga_description/urdf/beluga_base.xacro (robot description, xacro)
@@ -29,5 +29,5 @@
   <!-- minion_usv_height is not really! It's just for run... We need first calculate the Fossen parameters -->
   <!-- Volume -->
-  <xacro:property name="volume" value="0.0325"/>
+  <xacro:property name="volume" value="0.0305"/>
   <!-- Center of gravity -->
   <xacro:property name="cog" value="0 0 -0.08"/>
@@ -60,6 +60,6 @@
           <origin xyz="${cog}" rpy="0 0 0"/>
           <inertia
-            ixx="${0.503217}" ixy="${0.000204}" ixz="${-0.000526}"
-            iyy="${0.493449}" iyz="${0.000038}" izz="${0.919819}" />
+            ixx="${503.217}" ixy="${0.0}" ixz="${0.0}"
+            iyy="${493.449}" iyz="${0.0}" izz="${919.819}" />
         </inertial>
         <!-- This visual geometry representation can be used when running

Commit message: Changed parameters so it matches the values in beluga.yaml. Beluga 'tilts' quite a bit downwards in the simulator.

File: beluga_description/urdf/beluga_base.xacro (robot description, xacro)
@@ -22,14 +22,14 @@
   -->
   <!-- Mass -->
-  <xacro:property name="mass" value="30.9"/>
+  <xacro:property name="mass" value="24.00"/>
   <!-- Describing the dimensions of the vehicle's bounding box: width, length, height -->
-  <xacro:property name="x_size" value="0.400"/>
-  <xacro:property name="y_size" value="0.400"/>
-  <xacro:property name="z_size" value="0.20066"/>
+  <xacro:property name="x_size" value="0.367"/>
+  <xacro:property name="y_size" value="0.316"/>
+  <xacro:property name="z_size" value="0.216"/>
   <!-- minion_usv_height is not really! It's just for run... We need first calculate the Fossen parameters -->
   <!-- Volume -->
-  <xacro:property name="volume" value="0.0325"/>
+  <xacro:property name="volume" value="0.025"/>
   <!-- Center of gravity -->
-  <xacro:property name="cog" value="0 0 -0.08"/>
+  <xacro:property name="cog" value="-0.0152 0.001 0.0094"/>
   <!--
   Center of buoyancy according to eq. (3.1) p. 28 in Berg2012.
@@ -37,5 +37,5 @@
   assume NWU (otherwise cob is below cog?). 0.155
   -->
-  <xacro:property name="cob" value="0 0 0.05"/>
+  <xacro:property name="cob" value="-0.0151 0.0009 0.020"/>
   <!-- Fluid density -->
   <xacro:property name="rho" value="1028"/>
@@ -60,6 +60,6 @@
           <origin xyz="${cog}" rpy="0 0 0"/>
           <inertia
-            ixx="${0.503217}" ixy="${0.000204}" ixz="${-0.000526}"
-            iyy="${0.493449}" iyz="${0.000038}" izz="${0.919819}" />
+            ixx="${0.50}" ixy="${0.000204}" ixz="${-0.000526}"
+            iyy="${1.1}" iyz="${0.000038}" izz="${1.2}" />
         </inertial>
         <!-- This visual geometry representation can be used when running

Commit message: Updated the parameters again so that its identical to beluga.yaml. You can still drive the drone in the simulator with joystick, but the tuning is not good.

File: beluga_description/urdf/beluga_base.xacro (robot description, xacro)
@@ -24,10 +24,10 @@
   <xacro:property name="mass" value="24.00"/>
   <!-- Describing the dimensions of the vehicle's bounding box: width, length, height -->
-  <xacro:property name="x_size" value="0.367"/>
-  <xacro:property name="y_size" value="0.316"/>
-  <xacro:property name="z_size" value="0.216"/>
+  <xacro:property name="x_size" value="0.73"/>
+  <xacro:property name="y_size" value="0.63"/>
+  <xacro:property name="z_size" value="0.42"/>
   <!-- minion_usv_height is not really! It's just for run... We need first calculate the Fossen parameters -->
   <!-- Volume -->
-  <xacro:property name="volume" value="0.025"/>
+  <xacro:property name="volume" value="0.020"/>
   <!-- Center of gravity -->
   <xacro:property name="cog" value="-0.0152 0.001 0.0094"/>

Commit message: Calibrating the simulation parameters

File: beluga_description/urdf/beluga_base.xacro (robot description, xacro)
@@ -29,7 +29,7 @@
   <!-- minion_usv_height is not really! It's just for run... We need first calculate the Fossen parameters -->
   <!-- Volume -->
-  <xacro:property name="volume" value="0.020"/>
+  <xacro:property name="volume" value="0.0325"/>
   <!-- Center of gravity -->
-  <xacro:property name="cog" value="-0.0152 0.001 0.0094"/>
+  <xacro:property name="cog" value="0.0 0.0 -0.08"/> <!--0.0067-->
   <!--
   Center of buoyancy according to eq. (3.1) p. 28 in Berg2012.
@@ -37,5 +37,5 @@
   assume NWU (otherwise cob is below cog?). 0.155
   -->
-  <xacro:property name="cob" value="-0.0151 0.0009 0.020"/>
+  <xacro:property name="cob" value="0.0 0.0 0.05"/>
   <!-- Fluid density -->
   <xacro:property name="rho" value="1028"/>

Commit message: Changed the mass back to mantas simulator weight and changed the name manta_sensors to beluga_sensors

File: beluga_description/urdf/beluga_base.xacro (robot description, xacro)
@@ -22,5 +22,5 @@
   -->
   <!-- Mass -->
-  <xacro:property name="mass" value="24.00"/>
+  <xacro:property name="mass" value="30.9"/>
   <!-- Describing the dimensions of the vehicle's bounding box: width, length, height -->
   <xacro:property name="x_size" value="0.73"/>
@@ -63,9 +63,4 @@
             iyy="${1.1}" iyz="${0.000038}" izz="${1.2}" />
         </inertial>
-        <!-- This visual geometry representation can be used when running
-             tasks in which you need Gazebo to start quickly
-        -->
-        <!-- <xacro:if value="${use_simplified_mesh}"> -->
-        <!-- Code in rexrov2_base.xacro if use the flag use_simplified_mesh -->
         <visual>
           <origin xyz="0 0 0" rpy="0 0 0"/>
@@ -98,5 +93,5 @@
      This .xacro file has to run to be able to move the robot when controller
      commands have been sent to the thrusters-->
-  <xacro:include filename="$(find beluga_description)/urdf/manta_sensors.xacro"/>
+  <xacro:include filename="$(find beluga_description)/urdf/beluga_sensors.xacro"/>
   </xacro:macro>
   <gazebo reference="${namespace}/base_link">

Commit message: Changed x,y,z values back to manta values

File: beluga_description/urdf/beluga_base.xacro (robot description, xacro)
@@ -24,12 +24,12 @@
   <xacro:property name="mass" value="30.9"/>
   <!-- Describing the dimensions of the vehicle's bounding box: width, length, height -->
-  <xacro:property name="x_size" value="0.73"/>
-  <xacro:property name="y_size" value="0.63"/>
-  <xacro:property name="z_size" value="0.42"/>
+  <xacro:property name="x_size" value="0.400"/>
+  <xacro:property name="y_size" value="0.400"/>
+  <xacro:property name="z_size" value="0.20066"/>
   <!-- minion_usv_height is not really! It's just for run... We need first calculate the Fossen parameters -->
   <!-- Volume -->
   <xacro:property name="volume" value="0.0325"/>
   <!-- Center of gravity -->
-  <xacro:property name="cog" value="0.0 0.0 -0.08"/> <!--0.0067-->
+  <xacro:property name="cog" value="0.0 0.0 -0.08"/>
   <!--
   Center of buoyancy according to eq. (3.1) p. 28 in Berg2012.
@@ -60,6 +60,6 @@
           <origin xyz="${cog}" rpy="0 0 0"/>
           <inertia
-            ixx="${0.50}" ixy="${0.000204}" ixz="${-0.000526}"
-            iyy="${1.1}" iyz="${0.000038}" izz="${1.2}" />
+            ixx="${0.503217}" ixy="${0.000204}" ixz="${-0.000526}"
+            iyy="${0.493449}" iyz="${0.000038}" izz="${0.919819}" />
         </inertial>
         <visual>

Commit message: Simulator renaming from manta to beluga (#44)
* Changed from manta to beluga, not parameters.

* Changed parameters so it matches the values in beluga.yaml. Beluga 'tilts' quite a bit downwards in the simulator.

* Updated the parameters again so that its identical to beluga.yaml. You can still drive the drone in the simulator with joystick, but the tuning is not good.

* Calibrating the simulation parameters

* Changed the mass back to mantas simulator weight and changed the name manta_sensors to beluga_sensors

* Deleted manta_actuators from beluga_description since it was never used in this package for beluga. The same file, manta_actuators, is still in manta_description.

* Changed x,y,z values back to manta values

Co-authored-by: Torben Falleth Olsen <you@example.com>
Co-authored-by: simonvolden <simonvolden@gmail.com>

File: beluga_description/urdf/beluga_base.xacro (robot description, xacro)
@@ -14,5 +14,5 @@
   -->
   <!-- includes -->
-  <xacro:include filename="$(find manta_description)/urdf/common.urdf.xacro"/>
+  <xacro:include filename="$(find beluga_description)/urdf/common.urdf.xacro"/>
   <xacro:include filename="$(find uuv_sensor_ros_plugins)/urdf/sensor_snippets.xacro"/>
   <xacro:include filename="$(find uuv_gazebo_ros_plugins)/urdf/snippets.xacro"/>
@@ -31,5 +31,5 @@
   <xacro:property name="volume" value="0.0325"/>
   <!-- Center of gravity -->
-  <xacro:property name="cog" value="0 0 -0.08"/>
+  <xacro:property name="cog" value="0.0 0.0 -0.08"/>
   <!--
   Center of buoyancy according to eq. (3.1) p. 28 in Berg2012.
@@ -37,5 +37,5 @@
   assume NWU (otherwise cob is below cog?). 0.155
   -->
-  <xacro:property name="cob" value="0 0 0.05"/>
+  <xacro:property name="cob" value="0.0 0.0 0.05"/>
   <!-- Fluid density -->
   <xacro:property name="rho" value="1028"/>
@@ -63,9 +63,4 @@
             iyy="${0.493449}" iyz="${0.000038}" izz="${0.919819}" />
         </inertial>
-        <!-- This visual geometry representation can be used when running
-             tasks in which you need Gazebo to start quickly
-        -->
-        <!-- <xacro:if value="${use_simplified_mesh}"> -->
-        <!-- Code in rexrov2_base.xacro if use the flag use_simplified_mesh -->
         <visual>
           <origin xyz="0 0 0" rpy="0 0 0"/>
@@ -98,5 +93,5 @@
      This .xacro file has to run to be able to move the robot when controller
      commands have been sent to the thrusters-->
-  <xacro:include filename="$(find beluga_description)/urdf/manta_sensors.xacro"/>
+  <xacro:include filename="$(find beluga_description)/urdf/beluga_sensors.xacro"/>
   </xacro:macro>
   <gazebo reference="${namespace}/base_link">
