Commit message: add beluga mk2
Signed-off-by: Christopher Strøm <detoxte@gmail.com>

File: robots/beluga_description/urdf/beluga_base.xacro (robot description, xacro)
@@ -22,12 +22,12 @@
   -->
   <!-- Mass -->
-  <xacro:property name="mass" value="30.9"/>
+  <xacro:property name="mass" value="35.0"/>
   <!-- Describing the dimensions of the vehicle's bounding box: width, length, height -->
-  <xacro:property name="x_size" value="0.400"/>
+  <xacro:property name="x_size" value="0.800"/>
   <xacro:property name="y_size" value="0.400"/>
-  <xacro:property name="z_size" value="0.20066"/>
+  <xacro:property name="z_size" value="0.600"/>
   <!-- minion_usv_height is not really! It's just for run... We need first calculate the Fossen parameters -->
   <!-- Volume -->
-  <xacro:property name="volume" value="0.0325"/>
+  <xacro:property name="volume" value="0.0365"/>
   <!-- Center of gravity -->
   <xacro:property name="cog" value="0.0 0.0 -0.08"/>
@@ -48,5 +48,5 @@
   <!-- Parameters -->
   <xacro:property name="namespace" value="beluga"/>
-  <xacro:property name="visual_mesh_file" value="file://$(find beluga_description)/mesh/beluga_centered_body.dae"/>
+  <xacro:property name="visual_mesh_file" value="file://$(find beluga_description)/mesh/mk2.stl"/>
   <xacro:macro name="beluga_base" params="namespace *gazebo inertial_reference_frame">
    <!-- Rigid body description of the base link -->
@@ -64,7 +64,7 @@
         </inertial>
         <visual>
-          <origin xyz="0 0 0" rpy="0 0 0"/>
+          <origin xyz="0 0 0" rpy="0 0 1.57"/>
           <geometry>
-            <mesh filename="${visual_mesh_file}" scale="0.01 0.01 0.01" />
+            <mesh filename="${visual_mesh_file}" scale="1.0 1.0 1.0" />
           </geometry>
         </visual>

File: robots/beluga_description/urdf/beluga_sensors.xacro (robot description, xacro)
@@ -10,5 +10,5 @@
     parent_link="${namespace}/base_link"
     inertial_reference_frame="${inertial_reference_frame}">
-    <origin xyz="0.074 -0.015 -0.115" rpy="-3.14 1.57 -3.14"/>
+    <origin xyz="0.0 0.0 -0.135" rpy="-3.14 1.57 -3.14"/>
   </xacro:default_dvl_macro>
   <!-- Magnetometer  -->
@@ -35,12 +35,13 @@
   </xacro:default_imu_macro>
   <!-- Mount a camera -->
+  <!-- The front left camera is used for the CV pipeline -->
   <xacro:default_camera namespace="${namespace}" parent_link="${namespace}/base_link" suffix="front_left">
-    <origin xyz="0.349 0.1 0.058" rpy="0.00 0.0 0.0"/>
+    <origin xyz="0.4 0.05 0.025" rpy="0.00 0.0 0.0"/>
   </xacro:default_camera>
   <xacro:default_camera namespace="${namespace}" parent_link="${namespace}/base_link" suffix="front_right">
-    <origin xyz="0.349 -0.1 0.058" rpy="0.00 0.0 0.0"/>
+    <origin xyz="0.4 -0.05 0.025" rpy="0.00 0.0 0.0"/>
   </xacro:default_camera>
   <xacro:default_camera namespace="${namespace}" parent_link="${namespace}/base_link" suffix="under">
-    <origin xyz="0.15 0.0 -0.15" rpy="0 ${0.5*pi} 0"/>
+    <origin xyz="-0.025 -0.08 -0.17" rpy="0 ${0.5*pi} 0"/>
   </xacro:default_camera>
 <!--
